File: sensors.kicad_sch (KiCad schematic)
At the start: 20 parts, among them J3 Ultrasonic sensor, J4 AVR-ISP-6, J5 POT, SW1 Light control, U2 ATmega328P-P, Y1 16MHz

Commit message: Final schematic before layout
Parts:
- removed J3: Ultrasonic sensor, symbol Connector_Generic:Conn_01x04
- added C?: 1uF, Capacitor_SMD:C_0402_1005Metric, symbol Device:C
- added R?: 10k, Resistor_SMD:R_0603_1608Metric, symbol Device:R
- added U5: HC-SR04, footprints:XCVR_HC-SR04, symbol HC-SR04:HC-SR04
- C?: renamed from C3; footprint (none) -> Capacitor_SMD:C_0402_1005Metric
- C?: renamed from C6; footprint (none) -> Capacitor_SMD:C_0805_2012Metric
- C?: renamed from C2; footprint (none) -> Capacitor_SMD:C_0402_1005Metric
- C?: renamed from C4; footprint (none) -> Capacitor_SMD:C_0402_1005Metric
- C?: renamed from C5; footprint (none) -> Capacitor_SMD:C_0805_2012Metric
- J?: renamed from J5; footprint (none) -> Connector_Molex:Molex_KK-254_AE-6410-03A_1x03_P2.54mm_Vertical
- LED?: renamed from LED3; footprint ALS-DPDIC17-78C_L749_TR8:ALSDPDIC1778CL749TR8 -> footprints:ALSDPDIC1778CL749TR8
- LED?: renamed from LED2; footprint ALS-DPDIC17-78C_L749_TR8:ALSDPDIC1778CL749TR8 -> footprints:ALSDPDIC1778CL749TR8
- LED?: renamed from LED1; footprint ALS-DPDIC17-78C_L749_TR8:ALSDPDIC1778CL749TR8 -> footprints:ALSDPDIC1778CL749TR8
- LED?: renamed from LED4; footprint ALS-DPDIC17-78C_L749_TR8:ALSDPDIC1778CL749TR8 -> footprints:ALSDPDIC1778CL749TR8
- R?: renamed from R6; footprint (none) -> Resistor_SMD:R_0603_1608Metric
- R?: renamed from R4; footprint (none) -> Resistor_SMD:R_0603_1608Metric
- R?: renamed from R3; footprint (none) -> Resistor_SMD:R_0603_1608Metric
- R?: renamed from R5; footprint (none) -> Resistor_SMD:R_0603_1608Metric
- SW?: renamed from SW1; value Light control -> Override switch; footprint (none) -> Button_Switch_SMD:SW_SPST_CK_KXT3
- Y?: renamed from Y1; footprint (none) -> Crystal:Crystal_HC49-U_Vertical
- renumbered D1 to D?, J4 to J?, U2 to U?
Connections:
- net Power in is gone; now on net Flyback output: SW?.1
- net Echo: now also U5.3 (ECHO)
- net Flyback output: now also U5.1 (VCC)
- net GND: now also C?.2, U5.4 (GND)
- net Trig: now also U5.2 (TRIG)
- net Override signal: now reaches U?.3 (PD1)
- net Override signal: now also C?.1, R?.1
- net Power out: no longer names the net of SW?.2
- net Power out: now also R?.2
Other:
- moved on the sheet: SW?

Commit message: Almost done with sensors layout
Connections:
- net INT: now also U?.4 (PD2); no longer U?.14 (PB0)
- net Override signal: now also U?.25 (PC2); no longer U?.3 (PD1)
Changed lines of the file:
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@@
-    (stroke (width 0) (type default))
-  )
-  (wire (pts (xy 213.36 168.91) (xy 217.17 168.91))
     (stroke (width 0) (type default))
   )
@@
     (stroke (width 0) (type default))
   )
+  (wire (pts (xy 213.36 151.13) (xy 218.44 151.13))
+    (stroke (width 0) (type default))
+  )
   (wire (pts (xy 142.24 67.31) (xy 146.05 67.31))
     (stroke (width 0) (type default))
@@
     (stroke (width 0) (type default))
   )
-  (wire (pts (xy 213.36 123.19) (xy 218.44 123.19))
-    (stroke (width 0) (type default))
-  )
   (polyline (pts (xy 168.91 95.25) (xy 119.38 95.25))
     (stroke (width 0) (type dash))
@@
   )
   (wire (pts (xy 95.25 130.81) (xy 100.33 130.81))
+    (stroke (width 0) (type default))
+  )
+  (wire (pts (xy 213.36 171.45) (xy 218.44 171.45))
     (stroke (width 0) (type default))
   )
@@
     (effects (font (size 1.27 1.27)) (justify left bottom))
   )
-  (label "Override signal" (at 217.17 168.91 0) (fields_autoplaced)
+  (label "Override signal" (at 218.44 151.13 0) (fields_autoplaced)
     (effects (font (size 1.27 1.27)) (justify left bottom))
   )
@@
     (effects (font (size 1.27 1.27)) (justify left bottom))
   )
-  (label "INT" (at 218.44 123.19 0) (fields_autoplaced)
-    (effects (font (size 1.27 1.27)) (justify left bottom))
-  )
+  (label "INT" (at 218.44 171.45 0) (fields_autoplaced)
+    (effects (font (size 1.27 1.27)) (justify left bottom))
+  )
