File: pcb/445.kicad_sch (KiCad schematic)
At the start: 43 parts, among them Q1 Q_NPN_BCE, T1 Transformer_SP_1S, U1 UCC28720D, U2 TPS71533DCKR

Commit message: Restructure project repository
Parts:
- added TP6: TestPoint, TestPoint:TestPoint_Loop_D3.80mm_Drill2.0mm, symbol Connector:TestPoint
- J? (x2): footprint TerminalBlock_MetzConnect:TerminalBlock_MetzConnect_360410_1x01_Horizontal_ScrewM3.0 -> 445:MountingHole_8.0mm_M8_Pad_TopBottom
- Q1: footprint footprints:ALSDPDIC1778CL749TR8 -> Package_TO_SOT_THT:TO-92L
- R8: value 200 -> 330
- R?: value 100 -> 470
- R?: value 100 -> 360
- T1: footprint footprints:750317828 -> 445:750813314update
- TP1, TP2, TP3, TP4, TP5, TP8: footprint TestPoint:TestPoint_Loop_D3.80mm_Drill2.8mm -> TestPoint:TestPoint_Loop_D3.80mm_Drill2.0mm
Connections:
- net GND: no longer C?.2
- net at Q?.3 (G), U?.4: now also C?.2
- net at Q1.1 (B), U1.6 (DRV): now also TP6.1
Other:
- moved on the sheet: C?, R16
