File: pcb/sensors.kicad_sch (KiCad schematic)
At the start: 22 parts, among them U5 HC-SR04

Commit message: Restructure project repository
Parts:
- removed C? (x2): 1uF, Capacitor_SMD:C_0402_1005Metric, symbol Device:C
- removed LED? (x4): ALS-DPDIC17-78C_L749_TR8, footprints:ALSDPDIC1778CL749TR8, symbol ALS-DPDIC17-78C_L749_TR8:ALS-DPDIC17-78C_L749_TR8
- removed R?: 10k, Resistor_SMD:R_0603_1608Metric, symbol Device:R
- removed R? (x2): 1k, Resistor_SMD:R_0603_1608Metric, symbol Device:R
- added J3: Conn_01x10_Socket, Connector_PinSocket_2.54mm:PinSocket_1x10_P2.54mm_Vertical, symbol Connector:Conn_01x10_Socket
Connections:
- net 3.3V linear regulator output: now also J3.1 (Pin_1)
- net GND: now also J3.3 (Pin_3)
- net SCL: now also J3.4 (Pin_4)
- net SDA: now also J3.5 (Pin_5)
- net PD5: now reaches U?.11 (PD5)
- net PD5: now also J3.10 (Pin_10)
- net PD1: now reaches U?.3 (PD1)
- net PD1: now also J3.6 (Pin_6)
- net PD3: now reaches U?.5 (PD3)
- net PD3: now also J3.8 (Pin_8)
- net INT renamed PD2
- net PD2: now also J3.7 (Pin_7)
- new net 3Vo: J3.2 (Pin_2)
Other:
- note removed: "Luminosity sensors"
